Commit message: modifying the mass and inertia from the robot measurments

File: wsg_50_simulation/urdf/wsg_50.urdf.xacro (robot description, xacro)
@@ -9,24 +9,60 @@
                         Use e.g. for single contact point tip on finger. (default 0) -->
     <xacro:macro name="wsg_50_xacro" params="name parent finger_length finger_tip hardware_interface *origin">
-        <joint name="${name}_anterior_gripper_joint" type="fixed">
+        <joint name="${name}_plate_joint" type="fixed">
             <xacro:insert_block name="origin"/>
             <!-- <origin xyz="0 0 0" rpy="0 0 -1.5708"/> -->
             <parent link="${parent}"/>
-            <child link="${name}_base_link"/>
+            <child link="${name}_plate"/>
+        </joint>
+        <!-- GRIPPER PLATE -->
+        <link name="${name}_plate">
+          <inertial>
+            <mass value="0.0"/> <!-- This is not the true mass -->
+            <origin xyz="0 0 0"/>
+            <inertia ixx="1.0" ixy="0.0" ixz="0.0" iyy="1.0" iyz="0.0" izz="1.0"/> <!-- This are not the true inertia -->
+          </inertial>
+          <visual>
+            <origin rpy="0 0 0" xyz="0.0 0 0"/>
+            <geometry>
+              <mesh filename="package://med_description/meshes/wsg50/wsg50_plate.stl" scale="1 1 1"/>
+              <!--box size="0.146 0.05 0.0735"/-->
+            </geometry>
+            <material name="grey">
+              <color rgba="0.5 0.5 0.5 1"/>
+            </material>
+          </visual>
+          <collision>
+            <origin rpy="0 0 0" xyz="0.0 0 0"/>
+            <geometry>
+              <!--box size="0.146 0.05 0.0735"/-->
+              <mesh filename="package://med_description/meshes/wsg50/wsg50_plate.stl" scale="1 1 1"/>
+            </geometry>
+          </collision>
+        </link>
+        <gazebo reference="${name}_plate">
+          <material>Gazebo/Grey</material>
+          <turnGravityOff>false</turnGravityOff>
+        </gazebo>
+        <!-- GRIPPER -->
+        <joint name="${name}_anterior_gripper_joint" type="fixed">
+          <origin rpy="0 0 0" xyz="0 0 0.01"/>
+          <!-- <origin xyz="0 0 0" rpy="0 0 -1.5708"/> -->
+          <parent link="${name}_plate"/>
+          <child link="${name}_base_link"/>
         </joint>
         <!-- BASE LINK -->
         <link name="${name}_base_link">
             <inertial>
-                <mass value="0.25"/>
-                <origin xyz="0 0 0"/>
+                <mass value="1.48"/>
+                <origin xyz="0.00363 -0.00829 0.015"/>
                 <!--inertia ixx="1.0" ixy="0.0" ixz="0.0"
                     iyy="100.0" iyz="0.0"
                     izz="1.0" /-->
-                <inertia ixx="1.0" ixy="0.0" ixz="0.0" iyy="1.0" iyz="0.0" izz="1.0"/>
-            </inertial>
-            <visual>
-                <origin xyz="0.0 0 0" rpy="0 0 0"/>
-                <geometry>
-                    <mesh filename="package://wsg_50_simulation/meshes/WSG50_110.stl" scale="1 1 1"/>
+                <inertia ixx="0.0" ixy="0.0" ixz="0.0" iyy="0.0" iyz="0.0" izz="0.0"/>
+            </inertial>
+            <visual>
+                <origin xyz="0.0 0 0" rpy="0 0 0"/>
+                <geometry>
+                    <mesh filename="package://med_description/meshes/wsg50/WSG50_110.stl" scale="1 1 1"/>
                     <!--box size="0.146 0.05 0.0735"/-->
                 </geometry>
@@ -39,5 +75,5 @@
                 <geometry>
                     <!--box size="0.146 0.05 0.0735"/-->
-                    <mesh filename="package://wsg_50_simulation/meshes/WSG50_110.stl" scale="1 1 1"/>
+                    <mesh filename="package://med_description/meshes/wsg50/WSG50_110.stl" scale="1 1 1"/>
                 </geometry>
             </collision>
@@ -53,4 +89,8 @@
         </joint>
         <link name="${name}_center">
+            <inertial>
+                <mass value="0"/>
+                <inertia ixx="0"  ixy="0"  ixz="0" iyy="0" iyz="0" izz="0" />
+            </inertial>
         </link>
         <!-- GRIPPER LEFT -->
@@ -62,5 +102,4 @@
             <dynamics friction="100" damping="100"/>
             <axis xyz="1 0 0"/>
-            <limit effort="100" velocity="100"/>
         </joint>
         <transmission name="${name}_base_trans_left">
@@ -84,5 +123,5 @@
                 <origin xyz="0.0 0 0" rpy="0 0 0"/>
                 <geometry>
-                    <mesh filename="package://wsg_50_simulation/meshes/GUIDE_WSG50_110.stl" scale="0.001 0.001 0.001"/>
+                    <mesh filename="package://med_description/meshes/wsg50/GUIDE_WSG50_110.stl" scale="0.001 0.001 0.001"/>
                     <!--box size="0.0175 0.03 0.024"/-->
                 </geometry>
@@ -95,5 +134,5 @@
                 <geometry>
                     <!--box size="0.0175 0.03 0.024"/-->
-                    <mesh filename="package://wsg_50_simulation/meshes/GUIDE_WSG50_110.stl" scale="0.001 0.001 0.001"/>
+                    <mesh filename="package://med_description/meshes/wsg50/GUIDE_WSG50_110.stl" scale="0.001 0.001 0.001"/>
                 </geometry>
             </collision>
@@ -124,5 +163,5 @@
                 <origin xyz="0.0 0 0" rpy="0 0 0"/>
                 <geometry>
-                    <mesh filename="package://wsg_50_simulation/meshes/WSG-FMF.stl" scale="0.001 0.001 0.001"/>
+                    <mesh filename="package://med_description/meshes/wsg50/WSG-FMF.stl" scale="0.001 0.001 0.001"/>
                 </geometry>
                 <material name="black">
@@ -133,5 +172,5 @@
                 <origin xyz="0 0 0" rpy="0 0 0"/>
                 <geometry>
-                    <mesh filename="package://wsg_50_simulation/meshes/WSG-FMF.stl" scale="0.001 0.001 0.001"/>
+                    <mesh filename="package://med_description/meshes/wsg50/WSG-FMF.stl" scale="0.001 0.001 0.001"/>
                 </geometry>
             </collision>
@@ -150,5 +189,4 @@
             <axis xyz="-1 0 0"/>
             <dynamics friction="100" damping="100"/>
-            <limit effort="100" velocity="100"/>
         </joint>
         <transmission name="${name}_base_trans_right">
@@ -172,5 +210,5 @@
                 <origin xyz="0.0 0 0" rpy="0 0 0"/>
                 <geometry>
-                    <mesh filename="package://wsg_50_simulation/meshes/GUIDE_WSG50_110.stl" scale="0.001 0.001 0.001"/>
+                    <mesh filename="package://med_description/meshes/wsg50/GUIDE_WSG50_110.stl" scale="0.001 0.001 0.001"/>
                     <!--box size="0.0175 0.03 0.024"/-->
                 </geometry>
@@ -183,5 +221,5 @@
                 <geometry>
                     <!--box size="0.0175 0.03 0.024"/-->
-                    <mesh filename="package://wsg_50_simulation/meshes/GUIDE_WSG50_110.stl" scale="0.001 0.001 0.001"/>
+                    <mesh filename="package://med_description/meshes/wsg50/GUIDE_WSG50_110.stl" scale="0.001 0.001 0.001"/>
                 </geometry>
             </collision>
@@ -212,5 +250,5 @@
                 <origin xyz="0.0 0 0" rpy="0 0 0"/>
                 <geometry>
-                    <mesh filename="package://wsg_50_simulation/meshes/WSG-FMF.stl" scale="0.001 0.001 0.001"/>
+                    <mesh filename="package://med_description/meshes/wsg50/WSG-FMF.stl" scale="0.001 0.001 0.001"/>
                 </geometry>
                 <material name="black">
@@ -221,5 +259,5 @@
                 <origin xyz="0 0 0" rpy="0 0 0"/>
                 <geometry>
-                    <mesh filename="package://wsg_50_simulation/meshes/WSG-FMF.stl" scale="0.001 0.001 0.001"/>
+                    <mesh filename="package://med_description/meshes/wsg50/WSG-FMF.stl" scale="0.001 0.001 0.001"/>
                 </geometry>
             </collision>
@@ -230,4 +268,46 @@
             <turnGravityOff>false</turnGravityOff>
         </gazebo>
+        <!-- GRASP FRAME -->
+        <joint name="${name}_grasp_frame_fake_joint" type="fixed">
+          <origin rpy="0 0 0" xyz="0 0 0.144"/> <!-- May be worth considering the parameter finger_tip-->
+          <!-- <origin xyz="0 0 0" rpy="0 0 -1.5708"/> -->
+          <parent link="${name}_base_link"/>
+          <child link="grasp_frame"/>
+        </joint>
+        <link name="grasp_frame">
+          <inertial>
+            <mass value="0.0"/>
+            <origin xyz="0 0 0"/>
+            <inertia ixx="0.0" ixy="0.0" ixz="0.0" iyy="0.0" iyz="0.0" izz="0.0"/>
+          </inertial>
+        </link>
+        <!-- RIGHT FINGER TIP FRAME -->
+        <joint name="${name}_right_finger_tip_fake_joint" type="fixed">
+          <origin rpy="0 0 3.14159" xyz="0 0 0.121"/> <!-- May be worth considering the parameter finger_tip-->
+          <!-- <origin xyz="0 0 0" rpy="0 0 -1.5708"/> -->
+          <parent link="${name}_finger_right"/>
+          <child link="${name}_finger_right_tip"/>
+        </joint>
+        <link name="${name}_finger_right_tip">
+          <inertial>
+            <mass value="0.0"/>
+            <origin xyz="0 0 0"/>
+            <inertia ixx="0.0" ixy="0.0" ixz="0.0" iyy="0.0" iyz="0.0" izz="0.0"/>
+          </inertial>
+        </link>
+        <!-- LEFT FINGER TIP FRAME -->
+        <joint name="${name}_left_finger_tip_fake_joint" type="fixed">
+          <origin rpy="0 0 0" xyz="0 0 0.121"/> <!-- May be worth considering the parameter finger_tip-->
+          <!-- <origin xyz="0 0 0" rpy="0 0 -1.5708"/> -->
+          <parent link="${name}_finger_left"/>
+          <child link="${name}_finger_left_tip"/>
+        </joint>
+        <link name="${name}_finger_left_tip">
+          <inertial>
+            <mass value="0.0"/>
+            <origin xyz="0 0 0"/>
+            <inertia ixx="0.0" ixy="0.0" ixz="0.0" iyy="0.0" iyz="0.0" izz="0.0"/>
+          </inertial>
+        </link>
     </xacro:macro>
 </robot>
